File: v0.5/SMD/Latest/inputs.kicad_sch (KiCad schematic)
At the start: 44 parts, among them IC3 Trig Cond Socket, U5 MPX4250, U6 SP720

Commit message: placing components
Parts:
- U5: footprint Misc:MPX4250 -> Connector_PinHeader_2.54mm:PinHeader_1x06_P2.54mm_Horizontal
Changed lines of the file:
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@@
 (kicad_sch (version 20210621) (generator eeschema)
   (paper "A4")
+  (junction (at 59.69 128.27) (diameter 0) (color 0 0 0 0))
+  (junction (at 247.65 88.9) (diameter 0) (color 0 0 0 0))
+  (junction (at 156.21 95.25) (diameter 0) (color 0 0 0 0))
+  (junction (at 247.65 99.06) (diameter 0) (color 0 0 0 0))
+  (junction (at 208.28 106.68) (diameter 0) (color 0 0 0 0))
+  (junction (at 29.21 46.99) (diameter 0) (color 0 0 0 0))
+  (junction (at 82.55 48.26) (diameter 0) (color 0 0 0 0))
+  (junction (at 63.5 128.27) (diameter 0) (color 0 0 0 0))
+  (junction (at 68.58 128.27) (diameter 0) (color 0 0 0 0))
+  (junction (at 151.13 33.02) (diameter 0) (color 0 0 0 0))
+  (junction (at 41.91 128.27) (diameter 0) (color 0 0 0 0))
+  (junction (at 129.54 78.74) (diameter 0) (color 0 0 0 0))
+  (junction (at 86.36 48.26) (diameter 0) (color 0 0 0 0))
+  (junction (at 33.02 34.29) (diameter 0) (color 0 0 0 0))
+  (junction (at 247.65 105.41) (diameter 0) (color 0 0 0 0))
+  (junction (at 62.23 85.09) (diameter 0) (color 0 0 0 0))
+  (junction (at 208.28 99.06) (diameter 0) (color 0 0 0 0))
+  (junction (at 251.46 99.06) (diameter 0) (color 0 0 0 0))
+  (junction (at 156.21 49.53) (diameter 0) (color 0 0 0 0))
+  (junction (at 151.13 78.74) (diameter 0) (color 0 0 0 0))
+  (junction (at 129.54 33.02) (diameter 0) (color 0 0 0 0))
+  (junction (at 156.21 78.74) (diameter 0) (color 0 0 0 0))
+  (junction (at 251.46 105.41) (diameter 0) (color 0 0 0 0))
+  (junction (at 67.31 101.6) (diameter 0) (color 0 0 0 0))
+  (junction (at 130.81 125.73) (diameter 0) (color 0 0 0 0))
+  (junction (at 149.86 163.83) (diameter 0) (color 0 0 0 0))
+  (junction (at 73.66 41.91) (diameter 0) (color 0 0 0 0))
+  (junction (at 157.48 142.24) (diameter 0) (color 0 0 0 0))
+  (junction (at 40.64 85.09) (diameter 0) (color 0 0 0 0))
+  (junction (at 58.42 171.45) (diameter 0) (color 0 0 0 0))
+  (junction (at 67.31 85.09) (diameter 0) (color 0 0 0 0))
+  (junction (at 68.58 144.78) (diameter 0) (color 0 0 0 0))
+  (junction (at 157.48 125.73) (diameter 0) (color 0 0 0 0))
+  (junction (at 152.4 125.73) (diameter 0) (color 0 0 0 0))
+  (junction (at 53.34 171.45) (diameter 0) (color 0 0 0 0))
+  (junction (at 78.74 54.61) (diameter 0) (color 0 0 0 0))
+  (junction (at 41.91 144.78) (diameter 0) (color 0 0 0 0))
+  (junction (at 156.21 33.02) (diameter 0) (color 0 0 0 0))
   (junction (at 36.83 46.99) (diameter 0) (color 0 0 0 0))
-  (junction (at 68.58 128.27) (diameter 0) (color 0 0 0 0))
-  (junction (at 157.48 142.24) (diameter 0) (color 0 0 0 0))
-  (junction (at 149.86 163.83) (diameter 0) (color 0 0 0 0))
-  (junction (at 53.34 171.45) (diameter 0) (color 0 0 0 0))
-  (junction (at 59.69 128.27) (diameter 0) (color 0 0 0 0))
-  (junction (at 156.21 33.02) (diameter 0) (color 0 0 0 0))
-  (junction (at 157.48 125.73) (diameter 0) (color 0 0 0 0))
-  (junction (at 86.36 48.26) (diameter 0) (color 0 0 0 0))
-  (junction (at 62.23 85.09) (diameter 0) (color 0 0 0 0))
-  (junction (at 40.64 85.09) (diameter 0) (color 0 0 0 0))
-  (junction (at 152.4 125.73) (diameter 0) (color 0 0 0 0))
-  (junction (at 156.21 95.25) (diameter 0) (color 0 0 0 0))
-  (junction (at 68.58 144.78) (diameter 0) (color 0 0 0 0))
+  (junction (at 59.69 144.78) (diameter 0) (color 0 0 0 0))
   (junction (at 247.65 116.84) (diameter 0) (color 0 0 0 0))
-  (junction (at 156.21 78.74) (diameter 0) (color 0 0 0 0))
-  (junction (at 151.13 78.74) (diameter 0) (color 0 0 0 0))
-  (junction (at 82.55 48.26) (diameter 0) (color 0 0 0 0))
-  (junction (at 67.31 85.09) (diameter 0) (color 0 0 0 0))
-  (junction (at 247.65 88.9) (diameter 0) (color 0 0 0 0))
-  (junction (at 208.28 106.68) (diameter 0) (color 0 0 0 0))
-  (junction (at 63.5 128.27) (diameter 0) (color 0 0 0 0))
-  (junction (at 129.54 33.02) (diameter 0) (color 0 0 0 0))
-  (junction (at 41.91 128.27) (diameter 0) (color 0 0 0 0))
-  (junction (at 59.69 144.78) (diameter 0) (color 0 0 0 0))
-  (junction (at 247.65 99.06) (diameter 0) (color 0 0 0 0))
-  (junction (at 41.91 144.78) (diameter 0) (color 0 0 0 0))
-  (junction (at 251.46 105.41) (diameter 0) (color 0 0 0 0))
-  (junction (at 247.65 105.41) (diameter 0) (color 0 0 0 0))
-  (junction (at 78.74 54.61) (diameter 0) (color 0 0 0 0))
-  (junction (at 33.02 34.29) (diameter 0) (color 0 0 0 0))
-  (junction (at 156.21 49.53) (diameter 0) (color 0 0 0 0))
-  (junction (at 130.81 125.73) (diameter 0) (color 0 0 0 0))
-  (junction (at 151.13 33.02) (diameter 0) (color 0 0 0 0))
-  (junction (at 208.28 99.06) (diameter 0) (color 0 0 0 0))
-  (junction (at 58.42 171.45) (diameter 0) (color 0 0 0 0))
-  (junction (at 129.54 78.74) (diameter 0) (color 0 0 0 0))
-  (junction (at 67.31 101.6) (diameter 0) (color 0 0 0 0))
-  (junction (at 73.66 41.91) (diameter 0) (color 0 0 0 0))
-  (junction (at 251.46 99.06) (diameter 0) (color 0 0 0 0))
-  (junction (at 29.21 46.99) (diameter 0) (color 0 0 0 0))
   (wire (pts (xy 212.09 31.75) (xy 215.9 31.75))
     (stroke (width 0) (type default) (color 0 0 0 0))
@@
     )
   )
-  (symbol (lib_id "Misc:MPX4250") (at 50.8 48.26 0)
+  (symbol (lib_id "Misc:MPX4250") (at 50.8 48.26 0) (unit 1)
     (in_bom yes) (on_board yes)
     (property "Reference" "U5" (id 0) (at 50.165 40.7162 0)
@@
       (effects (font (size 1.524 1.524)))
     )
-    (property "Footprint" "Misc:MPX4250" (id 2) (at 49.53 48.26 0)
+    (property "Footprint" "Connector_PinHeader_2.54mm:PinHeader_1x06_P2.54mm_Horizontal" (id 2) (at 49.53 48.26 0)
       (effects (font (size 1.524 1.524)) hide)
     )
