File: v0.5/SMD/Latest/power.kicad_sch (KiCad schematic)
At the start: 13 parts, among them U8 LM2940S-5.0/NOPB

Commit message: placing components
Parts:
- C19: footprint Capacitor_SMD:C_0805_2012Metric_Pad1.15x1.40mm_HandSolder -> Capacitor_SMD:C_0805_2012Metric
- S1: footprint Misc:AYZ0202AGRLC -> SamacSys_Parts_github:AYZ0202AGRLC
Changed lines of the file:
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@@
 (kicad_sch (version 20210621) (generator eeschema)
   (paper "A4")
+  (junction (at 139.7 68.58) (diameter 0) (color 0 0 0 0))
+  (junction (at 180.34 62.23) (diameter 0) (color 0 0 0 0))
   (junction (at 161.29 78.74) (diameter 0) (color 0 0 0 0))
+  (junction (at 139.7 78.74) (diameter 0) (color 0 0 0 0))
+  (junction (at 175.26 78.74) (diameter 0) (color 0 0 0 0))
+  (junction (at 151.13 62.23) (diameter 0) (color 0 0 0 0))
+  (junction (at 128.27 78.74) (diameter 0) (color 0 0 0 0))
+  (junction (at 128.27 68.58) (diameter 0) (color 0 0 0 0))
+  (junction (at 184.15 68.58) (diameter 0) (color 0 0 0 0))
+  (junction (at 184.15 78.74) (diameter 0) (color 0 0 0 0))
   (junction (at 176.53 62.23) (diameter 0) (color 0 0 0 0))
-  (junction (at 180.34 62.23) (diameter 0) (color 0 0 0 0))
-  (junction (at 128.27 68.58) (diameter 0) (color 0 0 0 0))
-  (junction (at 128.27 78.74) (diameter 0) (color 0 0 0 0))
-  (junction (at 151.13 62.23) (diameter 0) (color 0 0 0 0))
-  (junction (at 184.15 68.58) (diameter 0) (color 0 0 0 0))
-  (junction (at 139.7 68.58) (diameter 0) (color 0 0 0 0))
   (junction (at 151.13 125.73) (diameter 0) (color 0 0 0 0))
-  (junction (at 139.7 78.74) (diameter 0) (color 0 0 0 0))
-  (junction (at 184.15 78.74) (diameter 0) (color 0 0 0 0))
-  (junction (at 175.26 78.74) (diameter 0) (color 0 0 0 0))
   (no_connect (at 213.36 55.88))
   (wire (pts (xy 138.43 125.73) (xy 140.97 125.73))
@@
     (pin "2")
   )
-  (symbol (lib_id "Device:D_Zener") (at 193.04 72.39 270)
+  (symbol (lib_id "Device:D_Zener") (at 193.04 72.39 270) (unit 1)
     (in_bom yes) (on_board yes)
     (property "Reference" "D15" (id 0) (at 195.0466 71.2216 90)
@@
     (property "Reference" "S1" (id 0) (at 166.37 121.539 0))
     (property "Value" "AYZ0202AGRLC" (id 1) (at 166.37 123.8504 0))
-    (property "Footprint" "Misc:AYZ0202AGRLC" (id 2) (at 176.53 125.73 0)
-      (effects (font (size 1.27 1.27)) (justify left) hide)
+    (property "Footprint" "SamacSys_Parts_github:AYZ0202AGRLC" (id 2) (at 176.53 125.73 0)
+      (effects (font (size 1.27 1.27)) (justify left))
     )
     (property "Datasheet" "" (id 3) (at 176.53 128.27 0)
@@
       (effects (font (size 1.27 1.27)) (justify left))
     )
-    (property "Footprint" "Capacitor_SMD:C_0805_2012Metric_Pad1.15x1.40mm_HandSolder" (id 2) (at 140.97 126.6952 0)
-      (effects (font (size 1.27 1.27)) hide)
-    )
+    (property "Footprint" "Capacitor_SMD:C_0805_2012Metric" (id 2) (at 140.97 126.6952 0)
+      (effects (font (size 1.27 1.27)) hide)
+    )
