File: v0.5/SMD/Latest/v0.4.4c.kicad_sch (KiCad schematic)
At the start: 1 part

Commit message: placing components
Parts:
- XA1: footprint Shields:Arduino_Mega2560_Shield_IO_Only -> Arduino:Arduino_Mega2560_Shield
Changed lines of the file:
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@@
   (paper "A4")
   (junction (at 114.3 123.19) (diameter 0) (color 0 0 0 0))
+  (junction (at 114.3 125.73) (diameter 0) (color 0 0 0 0))
+  (junction (at 114.3 120.65) (diameter 0) (color 0 0 0 0))
   (junction (at 120.65 135.89) (diameter 0) (color 0 0 0 0))
-  (junction (at 114.3 120.65) (diameter 0) (color 0 0 0 0))
-  (junction (at 114.3 125.73) (diameter 0) (color 0 0 0 0))
   (wire (pts (xy 186.69 135.89) (xy 189.23 135.89))
     (stroke (width 0) (type default) (color 0 0 0 0))
@@
       (effects (font (size 1.524 1.524)))
     )
-    (property "Footprint" "Shields:Arduino_Mega2560_Shield_IO_Only" (id 2) (at 171.45 16.51 0)
+    (property "Footprint" "Arduino:Arduino_Mega2560_Shield" (id 2) (at 171.45 16.51 0)
       (effects (font (size 1.524 1.524)) hide)
     )
@@
     )
     (path "/00000000-0000-0000-0000-00005cd18ec3/00000000-0000-0000-0000-00005cf0aad4"
-      (reference "C19") (unit 1) (value "22uF") (footprint "Capacitor_SMD:C_0805_2012Metric_Pad1.15x1.40mm_HandSolder")
+      (reference "C19") (unit 1) (value "22uF") (footprint "Capacitor_SMD:C_0805_2012Metric")
     )
     (path "/00000000-0000-0000-0000-00005cd18ec3/00000000-0000-0000-0000-00005cd284e9"
@@
     )
     (path "/00000000-0000-0000-0000-00005cd18ec3/00000000-0000-0000-0000-00005cddd447"
-      (reference "S1") (unit 1) (value "AYZ0202AGRLC") (footprint "Misc:AYZ0202AGRLC")
+      (reference "S1") (unit 1) (value "AYZ0202AGRLC") (footprint "SamacSys_Parts_github:AYZ0202AGRLC")
     )
     (path "/00000000-0000-0000-0000-00005cd18c17/00000000-0000-0000-0000-00005cd2eedb"
@@
     )
     (path "/00000000-0000-0000-0000-00005cd18d89/00000000-0000-0000-0000-00005cd196c6"
-      (reference "U5") (unit 1) (value "MPX4250") (footprint "Misc:MPX4250")
+      (reference "U5") (unit 1) (value "MPX4250") (footprint "Connector_PinHeader_2.54mm:PinHeader_1x06_P2.54mm_Horizontal")
     )
     (path "/00000000-0000-0000-0000-00005cd18d89/00000000-0000-0000-0000-00005cda8540"
@@
     )
     (path "/00000000-0000-0000-0000-00005cd14b53"
-      (reference "XA1") (unit 1) (value "Arduino_Mega2560_Shield") (footprint "Shields:Arduino_Mega2560_Shield_IO_Only")
-    )
-  )
+      (reference "XA1") (unit 1) (value "Arduino_Mega2560_Shield") (footprint "Arduino:Arduino_Mega2560_Shield")
+    )
+  )
