File: v0.5/SMD/Latest/v0.4.4c.kicad_pcb (KiCad board)
At the start: 2 copper layers, 100 x 100 mm, 299 parts, among them IC3 Trig Cond Socket, J1 Conn_01x05, J2 Conn_01x06, J3 Conn_01x02, J4 Conn_02x20_Counter_Clockwise, J5 Conn_01x04, J6 Conn_01x05, J7 Conn_01x05, J8 Conn_01x03, Q1 SSM3K357R, Q2 SSM3K357R, Q3 SSM3K357R, U1 VNLD5090, U2 TC4424A, U3 VNLD5090, U4 TC4424A, U5 MPX4250, U6 SP720, U7 VNLD5090, U8 LM2940S-5.0/NOPB, U9 VNLD5090

Commit message: placing components
Parts:
- removed G***: LOGO, Misc:WTM logo_sml
- removed REF** (x150): Pin_D1.0mm_L10.0mm, Connector_Pin:Pin_D1.0mm_L10.0mm
- C10, C13, C24, C25, C4, C7, D1, D17, D18, D2, D20, D3, D4, D5, D6, Q2, Q3, R1, R10, R11, R12, R13, R14, R2, R29, R3, R30, R32, R35, R39, R4, R47, R48, R49, R5, R50, R6, R7, R8, R9, U1, U2, U6, U7: moved to B.Cu
- C19: footprint Capacitor_SMD:C_0805_2012Metric_Pad1.15x1.40mm_HandSolder -> Capacitor_SMD:C_0805_2012Metric
- JP6, JP7, JP9: moved to F.Cu
- S1: footprint Misc:AYZ0202AGRLC -> SamacSys_Parts_github:AYZ0202AGRLC
- U5: footprint Misc:MPX4250 -> Connector_PinHeader_2.54mm:PinHeader_1x06_P2.54mm_Horizontal
- XA1: footprint Shields:Arduino_Mega2560_Shield_IO_Only -> Arduino:Arduino_Mega2560_Shield
- moved D13 234.6 mm to (-41.8, 129.0), turned to 0 degrees
- moved R37 222.7 mm to (-50.3, 126.3), turned to 0 degrees
- moved R33 202.5 mm to (243.2, -58.7), turned to 0 degrees
- moved C5 191.7 mm to (227.9, -56.5)
- moved C6 171.1 mm to (139.2, -39.0)
- moved R31 161.3 mm to (150.6, -29.9), turned to 0 degrees
- moved C3 159.1 mm to (141.7, -27.7)
- moved Q1 140.6 mm to (53.0, 11.6), turned to 0 degrees
- moved R51 139.0 mm to (48.7, 21.8), turned to 0 degrees
- moved R60 109.4 mm to (57.6, 13.8), turned to 0 degrees
- moved RV1 108.8 mm to (101.9, 104.5)
- moved C18 105.4 mm to (107.5, 114.1), turned to 180 degrees
- moved C17 103.9 mm to (111.8, 110.7), turned to -90 degrees
- moved D14 97.2 mm to (107.5, 105.3), turned to -90 degrees
- moved J3 90.7 mm to (116.2, 30.7), turned to -90 degrees
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Connections:
- A1 pad 10: Net-(A1-Pad10) -> unconnected-(A1-Pad10)
- A1 pad 11: Net-(A1-Pad11) -> unconnected-(A1-Pad11)
- A1 pad 12: Net-(A1-Pad12) -> unconnected-(A1-Pad12)
- A1 pad 2: Net-(A1-Pad2) -> unconnected-(A1-Pad2)
- J2 pad 6: Net-(J2-Pad6) -> unconnected-(J2-Pad6)
- S1 pad 4: Net-(S1-Pad4) -> unconnected-(S1-Pad4)
- S1 pad 5: Net-(S1-Pad5) -> unconnected-(S1-Pad5)
- S1 pad 6: Net-(S1-Pad6) -> unconnected-(S1-Pad6)
- U1 pad 2: Net-(U1-Pad2) -> unconnected-(U1-Pad2)
- U1 pad 4: Net-(U1-Pad4) -> unconnected-(U1-Pad4)
- U2 pad 1: Net-(U2-Pad1) -> unconnected-(U2-Pad1)
- U2 pad 8: Net-(U2-Pad8) -> unconnected-(U2-Pad8)
- U3 pad 2: Net-(U3-Pad2) -> unconnected-(U3-Pad2)
- U3 pad 4: Net-(U3-Pad4) -> unconnected-(U3-Pad4)
- U4 pad 1: Net-(U4-Pad1) -> unconnected-(U4-Pad1)
- U4 pad 8: Net-(U4-Pad8) -> unconnected-(U4-Pad8)
- U7 pad 2: Net-(U7-Pad2) -> unconnected-(U7-Pad2)
- U7 pad 4: Net-(U7-Pad4) -> unconnected-(U7-Pad4)
- U9 pad 2: Net-(U9-Pad2) -> unconnected-(U9-Pad2)
- U9 pad 4: Net-(U9-Pad4) -> unconnected-(U9-Pad4)
- XA1 pad 3V3: Net-(XA1-Pad3V3) -> unconnected-(XA1-Pad3V3)
- XA1 pad A11: Net-(XA1-PadA11) -> unconnected-(XA1-PadA11)
- XA1 pad A12: Net-(XA1-PadA12) -> unconnected-(XA1-PadA12)
- XA1 pad A13: Net-(XA1-PadA13) -> unconnected-(XA1-PadA13)
- XA1 pad A14: Net-(XA1-PadA14) -> unconnected-(XA1-PadA14)
- XA1 pad A15: Net-(XA1-PadA15) -> unconnected-(XA1-PadA15)
- XA1 pad AREF: Net-(XA1-PadAREF) -> unconnected-(XA1-PadAREF)
- XA1 pad IORF: Net-(XA1-PadIORF) -> unconnected-(XA1-PadIORF)
- XA1 pad SCL: Net-(XA1-PadSCL) -> unconnected-(XA1-PadSCL)
- XA1 pad SDA: Net-(XA1-PadSDA) -> unconnected-(XA1-PadSDA)
- XA1 pad VIN: Net-(XA1-PadVIN) -> unconnected-(XA1-PadVIN)
Routing:
- net VDD: track 347.1 -> 28.0 mm, vias 5 -> 0
- net 12V-SW: track 269.2 -> 25.7 mm, vias 4 -> 0
- net ADC-Clamp-10: track 201.7 -> 0.00 mm, vias 4 -> 0
- net VDDA: track 136.4 -> 4.67 mm
- net ADC-Clamp-8: track 145.2 -> 20.1 mm, vias 1 -> 0
- net ADC-Clamp-9: track 126.3 -> 12.7 mm, vias 1 -> 0
- net VR2-: track 84.8 -> 0.00 mm, vias 1 -> 0
- net VR1-: track 77.9 -> 0.00 mm, vias 1 -> 0
- net CRANK-IN: track 75.5 -> 4.31 mm, vias 2 -> 0
- net MCU-D47: track 69.0 -> 0.00 mm, vias 1 -> 0
- net MCU-D45: track 66.2 -> 0.00 mm, vias 1 -> 0
- net Net-(JP11-Pad2): track 70.3 -> 4.76 mm, vias 1 -> 0
- net CAM-IN: track 66.7 -> 4.21 mm, vias 2 -> 0
- net MCU-D24: track 61.8 -> 0.00 mm, vias 1 -> 0
- net Net-(R6-Pad1): track 64.0 -> 2.23 mm
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- removed copper zone on B.Cu, net GND
- removed copper zone on F.Cu, net GND
Other:
- board size 100 x 100 mm -> 121.8 x 77.2 mm
- net class Default removed
- board text removed: "1"
- board text removed: "12V"
- board text removed: "2"
- board text removed: "3"
- board text removed: "4"
- board text removed: "5V"
- board text removed: "A10"
- board text removed: "A9"
- board text removed: "ALIGN"
- board text removed: "BLUETOOTH"
- board text removed: "D21"
- board text removed: "DIRECT/TSC"
- board text removed: "GND"
- board text removed: "IGNITER"
- board text removed: "IGNITION CHANNEL"
- board text removed: "INJECTOR CHANNEL"
- board text removed: "MODULE CHIP THIS END"
- board text removed: "MOUNT FLAT SIDE UP"
- board text removed: "PRIMARY"
- board text removed: "PULL -UP"
- board text removed: "Prog"
- board text removed: "RESET CONTROL"
- board text removed: "RX"
- board text removed: "Run"
- board text removed: "SECONDARY"
- board text removed: "STEPPER IDLE DRV8825"
- board text removed: "Speeduino Community"
- board text removed: "Speeduino v0.4.4c"
- board text removed: "TRIGGER SETUP"
- board text removed: "TRIGGER SIGNAL CONDITIONER SOCKET"
- board text removed: "TX"
- board text removed: "VSS"
- board text removed: "© Josh Stewart &"

Commit message: adaptater
Parts:
- added G***: LOGO, Misc:WTM logo_sml, F.Cu at (202.5, 132.5)
- added REF**: Pin_D1.0mm_L10.0mm, Connector_Pin:Pin_D1.0mm_L10.0mm, F.Cu at (195.7, 86.5)
- added REF**: Pin_D1.0mm_L10.0mm, Connector_Pin:Pin_D1.0mm_L10.0mm, F.Cu at (172.9, 86.5)
- added REF**: Pin_D1.0mm_L10.0mm, Connector_Pin:Pin_D1.0mm_L10.0mm, F.Cu at (172.9, 71.2)
- added REF**: Pin_D1.0mm_L10.0mm, Connector_Pin:Pin_D1.0mm_L10.0mm, F.Cu at (170.3, 71.2)
- added REF**: Pin_D1.0mm_L10.0mm, Connector_Pin:Pin_D1.0mm_L10.0mm, F.Cu at (167.8, 71.2)
- added REF**: Pin_D1.0mm_L10.0mm, Connector_Pin:Pin_D1.0mm_L10.0mm, F.Cu at (165.2, 71.2)
- added REF**: Pin_D1.0mm_L10.0mm, Connector_Pin:Pin_D1.0mm_L10.0mm, F.Cu at (162.7, 71.2)
- added REF**: Pin_D1.0mm_L10.0mm, Connector_Pin:Pin_D1.0mm_L10.0mm, F.Cu at (160.2, 71.2)
- added REF**: Pin_D1.0mm_L10.0mm, Connector_Pin:Pin_D1.0mm_L10.0mm, F.Cu at (195.7, 68.7)
- added REF**: Pin_D1.0mm_L10.0mm, Connector_Pin:Pin_D1.0mm_L10.0mm, F.Cu at (193.2, 68.7)
- added REF**: Pin_D1.0mm_L10.0mm, Connector_Pin:Pin_D1.0mm_L10.0mm, F.Cu at (190.6, 68.7)
- added REF**: Pin_D1.0mm_L10.0mm, Connector_Pin:Pin_D1.0mm_L10.0mm, F.Cu at (188.1, 68.7)
- added REF**: Pin_D1.0mm_L10.0mm, Connector_Pin:Pin_D1.0mm_L10.0mm, F.Cu at (170.3, 86.5)
- added REF**: Pin_D1.0mm_L10.0mm, Connector_Pin:Pin_D1.0mm_L10.0mm, F.Cu at (185.6, 68.7)
- added REF**: Pin_D1.0mm_L10.0mm, Connector_Pin:Pin_D1.0mm_L10.0mm, F.Cu at (183.0, 68.7)
- added REF**: Pin_D1.0mm_L10.0mm, Connector_Pin:Pin_D1.0mm_L10.0mm, F.Cu at (180.5, 68.7)
- added REF**: Pin_D1.0mm_L10.0mm, Connector_Pin:Pin_D1.0mm_L10.0mm, F.Cu at (177.9, 68.7)
- added REF**: Pin_D1.0mm_L10.0mm, Connector_Pin:Pin_D1.0mm_L10.0mm, F.Cu at (175.4, 68.7)
- added REF**: Pin_D1.0mm_L10.0mm, Connector_Pin:Pin_D1.0mm_L10.0mm, F.Cu at (172.9, 68.7)
- added REF**: Pin_D1.0mm_L10.0mm, Connector_Pin:Pin_D1.0mm_L10.0mm, F.Cu at (170.3, 68.7)
- added REF**: Pin_D1.0mm_L10.0mm, Connector_Pin:Pin_D1.0mm_L10.0mm, F.Cu at (167.8, 68.7)
- added REF**: Pin_D1.0mm_L10.0mm, Connector_Pin:Pin_D1.0mm_L10.0mm, F.Cu at (165.2, 68.7)
- added REF**: Pin_D1.0mm_L10.0mm, Connector_Pin:Pin_D1.0mm_L10.0mm, F.Cu at (162.7, 68.7)
- added REF**: Pin_D1.0mm_L10.0mm, Connector_Pin:Pin_D1.0mm_L10.0mm, F.Cu at (167.8, 86.5)
- added REF**: Pin_D1.0mm_L10.0mm, Connector_Pin:Pin_D1.0mm_L10.0mm, F.Cu at (160.2, 68.7)
- added REF**: Pin_D1.0mm_L10.0mm, Connector_Pin:Pin_D1.0mm_L10.0mm, F.Cu at (195.7, 66.2)
- added REF**: Pin_D1.0mm_L10.0mm, Connector_Pin:Pin_D1.0mm_L10.0mm, F.Cu at (193.2, 66.2)
- added REF**: Pin_D1.0mm_L10.0mm, Connector_Pin:Pin_D1.0mm_L10.0mm, F.Cu at (190.6, 66.2)
- added REF**: Pin_D1.0mm_L10.0mm, Connector_Pin:Pin_D1.0mm_L10.0mm, F.Cu at (188.1, 66.2)
- added REF**: Pin_D1.0mm_L10.0mm, Connector_Pin:Pin_D1.0mm_L10.0mm, F.Cu at (185.6, 66.2)
- added REF**: Pin_D1.0mm_L10.0mm, Connector_Pin:Pin_D1.0mm_L10.0mm, F.Cu at (183.0, 66.2)
- added REF**: Pin_D1.0mm_L10.0mm, Connector_Pin:Pin_D1.0mm_L10.0mm, F.Cu at (180.5, 66.2)
- added REF**: Pin_D1.0mm_L10.0mm, Connector_Pin:Pin_D1.0mm_L10.0mm, F.Cu at (177.9, 66.2)
- added REF**: Pin_D1.0mm_L10.0mm, Connector_Pin:Pin_D1.0mm_L10.0mm, F.Cu at (175.4, 66.2)
- added REF**: Pin_D1.0mm_L10.0mm, Connector_Pin:Pin_D1.0mm_L10.0mm, F.Cu at (165.2, 86.5)
- added REF**: Pin_D1.0mm_L10.0mm, Connector_Pin:Pin_D1.0mm_L10.0mm, F.Cu at (172.9, 66.2)
- added REF**: Pin_D1.0mm_L10.0mm, Connector_Pin:Pin_D1.0mm_L10.0mm, F.Cu at (170.3, 66.2)
- added REF**: Pin_D1.0mm_L10.0mm, Connector_Pin:Pin_D1.0mm_L10.0mm, F.Cu at (167.8, 66.2)
- added REF**: Pin_D1.0mm_L10.0mm, Connector_Pin:Pin_D1.0mm_L10.0mm, F.Cu at (165.2, 66.2)
- added REF**: Pin_D1.0mm_L10.0mm, Connector_Pin:Pin_D1.0mm_L10.0mm, F.Cu at (162.7, 66.2)
- added REF**: Pin_D1.0mm_L10.0mm, Connector_Pin:Pin_D1.0mm_L10.0mm, F.Cu at (160.2, 66.2)
- added REF**: Pin_D1.0mm_L10.0mm, Connector_Pin:Pin_D1.0mm_L10.0mm, F.Cu at (195.7, 63.6)
- added REF**: Pin_D1.0mm_L10.0mm, Connector_Pin:Pin_D1.0mm_L10.0mm, F.Cu at (193.2, 63.6)
- added REF**: Pin_D1.0mm_L10.0mm, Connector_Pin:Pin_D1.0mm_L10.0mm, F.Cu at (190.6, 63.6)
- added REF**: Pin_D1.0mm_L10.0mm, Connector_Pin:Pin_D1.0mm_L10.0mm, F.Cu at (188.1, 63.6)
- added REF**: Pin_D1.0mm_L10.0mm, Connector_Pin:Pin_D1.0mm_L10.0mm, F.Cu at (162.7, 86.5)
- added REF**: Pin_D1.0mm_L10.0mm, Connector_Pin:Pin_D1.0mm_L10.0mm, F.Cu at (185.6, 63.6)
- added REF**: Pin_D1.0mm_L10.0mm, Connector_Pin:Pin_D1.0mm_L10.0mm, F.Cu at (183.0, 63.6)
- added REF**: Pin_D1.0mm_L10.0mm, Connector_Pin:Pin_D1.0mm_L10.0mm, F.Cu at (180.5, 63.6)
- added REF**: Pin_D1.0mm_L10.0mm, Connector_Pin:Pin_D1.0mm_L10.0mm, F.Cu at (177.9, 63.6)
- added REF**: Pin_D1.0mm_L10.0mm, Connector_Pin:Pin_D1.0mm_L10.0mm, F.Cu at (175.4, 63.6)
- added REF**: Pin_D1.0mm_L10.0mm, Connector_Pin:Pin_D1.0mm_L10.0mm, F.Cu at (172.9, 63.6)
- added REF**: Pin_D1.0mm_L10.0mm, Connector_Pin:Pin_D1.0mm_L10.0mm, F.Cu at (170.3, 63.6)
- added REF**: Pin_D1.0mm_L10.0mm, Connector_Pin:Pin_D1.0mm_L10.0mm, F.Cu at (167.8, 63.6)
- added REF**: Pin_D1.0mm_L10.0mm, Connector_Pin:Pin_D1.0mm_L10.0mm, F.Cu at (165.2, 63.6)
- added REF**: Pin_D1.0mm_L10.0mm, Connector_Pin:Pin_D1.0mm_L10.0mm, F.Cu at (162.7, 63.6)
- added REF**: Pin_D1.0mm_L10.0mm, Connector_Pin:Pin_D1.0mm_L10.0mm, F.Cu at (160.2, 86.5)
- added REF**: Pin_D1.0mm_L10.0mm, Connector_Pin:Pin_D1.0mm_L10.0mm, F.Cu at (160.2, 63.6)
- added REF**: Pin_D1.0mm_L10.0mm, Connector_Pin:Pin_D1.0mm_L10.0mm, F.Cu at (195.7, 83.9)
- added REF**: Pin_D1.0mm_L10.0mm, Connector_Pin:Pin_D1.0mm_L10.0mm, F.Cu at (193.2, 83.9)
- added REF**: Pin_D1.0mm_L10.0mm, Connector_Pin:Pin_D1.0mm_L10.0mm, F.Cu at (190.6, 83.9)
- added REF**: Pin_D1.0mm_L10.0mm, Connector_Pin:Pin_D1.0mm_L10.0mm, F.Cu at (188.1, 83.9)
- added REF**: Pin_D1.0mm_L10.0mm, Connector_Pin:Pin_D1.0mm_L10.0mm, F.Cu at (193.2, 86.5)
- added REF**: Pin_D1.0mm_L10.0mm, Connector_Pin:Pin_D1.0mm_L10.0mm, F.Cu at (185.6, 83.9)
- added REF**: Pin_D1.0mm_L10.0mm, Connector_Pin:Pin_D1.0mm_L10.0mm, F.Cu at (183.0, 83.9)
- added REF**: Pin_D1.0mm_L10.0mm, Connector_Pin:Pin_D1.0mm_L10.0mm, F.Cu at (180.5, 83.9)
- added REF**: Pin_D1.0mm_L10.0mm, Connector_Pin:Pin_D1.0mm_L10.0mm, F.Cu at (177.9, 83.9)
- added REF**: Pin_D1.0mm_L10.0mm, Connector_Pin:Pin_D1.0mm_L10.0mm, F.Cu at (175.4, 83.9)
- added REF**: Pin_D1.0mm_L10.0mm, Connector_Pin:Pin_D1.0mm_L10.0mm, F.Cu at (172.9, 83.9)
- added REF**: Pin_D1.0mm_L10.0mm, Connector_Pin:Pin_D1.0mm_L10.0mm, F.Cu at (170.3, 83.9)
- added REF**: Pin_D1.0mm_L10.0mm, Connector_Pin:Pin_D1.0mm_L10.0mm, F.Cu at (167.8, 83.9)
- added REF**: Pin_D1.0mm_L10.0mm, Connector_Pin:Pin_D1.0mm_L10.0mm, F.Cu at (165.2, 83.9)
- added REF**: Pin_D1.0mm_L10.0mm, Connector_Pin:Pin_D1.0mm_L10.0mm, F.Cu at (162.7, 83.9)
- added REF**: Pin_D1.0mm_L10.0mm, Connector_Pin:Pin_D1.0mm_L10.0mm, F.Cu at (190.6, 86.5)
- added REF**: Pin_D1.0mm_L10.0mm, Connector_Pin:Pin_D1.0mm_L10.0mm, F.Cu at (160.2, 83.9)
- added REF**: Pin_D1.0mm_L10.0mm, Connector_Pin:Pin_D1.0mm_L10.0mm, F.Cu at (195.7, 81.4)
- added REF**: Pin_D1.0mm_L10.0mm, Connector_Pin:Pin_D1.0mm_L10.0mm, F.Cu at (193.2, 81.4)
- added REF**: Pin_D1.0mm_L10.0mm, Connector_Pin:Pin_D1.0mm_L10.0mm, F.Cu at (190.6, 81.4)
- added REF**: Pin_D1.0mm_L10.0mm, Connector_Pin:Pin_D1.0mm_L10.0mm, F.Cu at (188.1, 81.4)
- added REF**: Pin_D1.0mm_L10.0mm, Connector_Pin:Pin_D1.0mm_L10.0mm, F.Cu at (185.6, 81.4)
- added REF**: Pin_D1.0mm_L10.0mm, Connector_Pin:Pin_D1.0mm_L10.0mm, F.Cu at (183.0, 81.4)
- added REF**: Pin_D1.0mm_L10.0mm, Connector_Pin:Pin_D1.0mm_L10.0mm, F.Cu at (180.5, 81.4)
- added REF**: Pin_D1.0mm_L10.0mm, Connector_Pin:Pin_D1.0mm_L10.0mm, F.Cu at (177.9, 81.4)
- added REF**: Pin_D1.0mm_L10.0mm, Connector_Pin:Pin_D1.0mm_L10.0mm, F.Cu at (175.4, 81.4)
- added REF**: Pin_D1.0mm_L10.0mm, Connector_Pin:Pin_D1.0mm_L10.0mm, F.Cu at (188.1, 86.5)
- added REF**: Pin_D1.0mm_L10.0mm, Connector_Pin:Pin_D1.0mm_L10.0mm, F.Cu at (172.9, 81.4)
- added REF**: Pin_D1.0mm_L10.0mm, Connector_Pin:Pin_D1.0mm_L10.0mm, F.Cu at (170.3, 81.4)
- added REF**: Pin_D1.0mm_L10.0mm, Connector_Pin:Pin_D1.0mm_L10.0mm, F.Cu at (167.8, 81.4)
- added REF**: Pin_D1.0mm_L10.0mm, Connector_Pin:Pin_D1.0mm_L10.0mm, F.Cu at (165.2, 81.4)
- added REF**: Pin_D1.0mm_L10.0mm, Connector_Pin:Pin_D1.0mm_L10.0mm, F.Cu at (162.7, 81.4)
- added REF**: Pin_D1.0mm_L10.0mm, Connector_Pin:Pin_D1.0mm_L10.0mm, F.Cu at (160.2, 81.4)
- added REF**: Pin_D1.0mm_L10.0mm, Connector_Pin:Pin_D1.0mm_L10.0mm, F.Cu at (195.7, 78.9)
- added REF**: Pin_D1.0mm_L10.0mm, Connector_Pin:Pin_D1.0mm_L10.0mm, F.Cu at (193.2, 78.9)
- added REF**: Pin_D1.0mm_L10.0mm, Connector_Pin:Pin_D1.0mm_L10.0mm, F.Cu at (190.6, 78.9)
- added REF**: Pin_D1.0mm_L10.0mm, Connector_Pin:Pin_D1.0mm_L10.0mm, F.Cu at (188.1, 78.9)
- added REF**: Pin_D1.0mm_L10.0mm, Connector_Pin:Pin_D1.0mm_L10.0mm, F.Cu at (185.6, 86.5)
- added REF**: Pin_D1.0mm_L10.0mm, Connector_Pin:Pin_D1.0mm_L10.0mm, F.Cu at (185.6, 78.9)
- added REF**: Pin_D1.0mm_L10.0mm, Connector_Pin:Pin_D1.0mm_L10.0mm, F.Cu at (183.0, 78.9)
- added REF**: Pin_D1.0mm_L10.0mm, Connector_Pin:Pin_D1.0mm_L10.0mm, F.Cu at (180.5, 78.9)
- added REF**: Pin_D1.0mm_L10.0mm, Connector_Pin:Pin_D1.0mm_L10.0mm, F.Cu at (177.9, 78.9)
- added REF**: Pin_D1.0mm_L10.0mm, Connector_Pin:Pin_D1.0mm_L10.0mm, F.Cu at (175.4, 78.9)
- added REF**: Pin_D1.0mm_L10.0mm, Connector_Pin:Pin_D1.0mm_L10.0mm, F.Cu at (172.9, 78.9)
- added REF**: Pin_D1.0mm_L10.0mm, Connector_Pin:Pin_D1.0mm_L10.0mm, F.Cu at (170.3, 78.9)
- added REF**: Pin_D1.0mm_L10.0mm, Connector_Pin:Pin_D1.0mm_L10.0mm, F.Cu at (167.8, 78.9)
- added REF**: Pin_D1.0mm_L10.0mm, Connector_Pin:Pin_D1.0mm_L10.0mm, F.Cu at (165.2, 78.9)
- added REF**: Pin_D1.0mm_L10.0mm, Connector_Pin:Pin_D1.0mm_L10.0mm, F.Cu at (162.7, 78.9)
- added REF**: Pin_D1.0mm_L10.0mm, Connector_Pin:Pin_D1.0mm_L10.0mm, F.Cu at (183.0, 86.5)
- added REF**: Pin_D1.0mm_L10.0mm, Connector_Pin:Pin_D1.0mm_L10.0mm, F.Cu at (160.2, 78.9)
- added REF**: Pin_D1.0mm_L10.0mm, Connector_Pin:Pin_D1.0mm_L10.0mm, F.Cu at (195.7, 76.3)
- added REF**: Pin_D1.0mm_L10.0mm, Connector_Pin:Pin_D1.0mm_L10.0mm, F.Cu at (193.2, 76.3)
- added REF**: Pin_D1.0mm_L10.0mm, Connector_Pin:Pin_D1.0mm_L10.0mm, F.Cu at (190.6, 76.3)
- added REF**: Pin_D1.0mm_L10.0mm, Connector_Pin:Pin_D1.0mm_L10.0mm, F.Cu at (188.1, 76.3)
- added REF**: Pin_D1.0mm_L10.0mm, Connector_Pin:Pin_D1.0mm_L10.0mm, F.Cu at (185.6, 76.3)
- added REF**: Pin_D1.0mm_L10.0mm, Connector_Pin:Pin_D1.0mm_L10.0mm, F.Cu at (183.0, 76.3)
- added REF**: Pin_D1.0mm_L10.0mm, Connector_Pin:Pin_D1.0mm_L10.0mm, F.Cu at (180.5, 76.3)
- added REF**: Pin_D1.0mm_L10.0mm, Connector_Pin:Pin_D1.0mm_L10.0mm, F.Cu at (177.9, 76.3)
- added REF**: Pin_D1.0mm_L10.0mm, Connector_Pin:Pin_D1.0mm_L10.0mm, F.Cu at (175.4, 76.3)
- added REF**: Pin_D1.0mm_L10.0mm, Connector_Pin:Pin_D1.0mm_L10.0mm, F.Cu at (180.5, 86.5)
- added REF**: Pin_D1.0mm_L10.0mm, Connector_Pin:Pin_D1.0mm_L10.0mm, F.Cu at (172.9, 76.3)
- added REF**: Pin_D1.0mm_L10.0mm, Connector_Pin:Pin_D1.0mm_L10.0mm, F.Cu at (170.3, 76.3)
- added REF**: Pin_D1.0mm_L10.0mm, Connector_Pin:Pin_D1.0mm_L10.0mm, F.Cu at (167.8, 76.3)
- added REF**: Pin_D1.0mm_L10.0mm, Connector_Pin:Pin_D1.0mm_L10.0mm, F.Cu at (165.2, 76.3)
- added REF**: Pin_D1.0mm_L10.0mm, Connector_Pin:Pin_D1.0mm_L10.0mm, F.Cu at (162.7, 76.3)
- added REF**: Pin_D1.0mm_L10.0mm, Connector_Pin:Pin_D1.0mm_L10.0mm, F.Cu at (160.2, 76.3)
- added REF**: Pin_D1.0mm_L10.0mm, Connector_Pin:Pin_D1.0mm_L10.0mm, F.Cu at (195.7, 73.8)
- added REF**: Pin_D1.0mm_L10.0mm, Connector_Pin:Pin_D1.0mm_L10.0mm, F.Cu at (193.2, 73.8)
- added REF**: Pin_D1.0mm_L10.0mm, Connector_Pin:Pin_D1.0mm_L10.0mm, F.Cu at (190.6, 73.8)
- added REF**: Pin_D1.0mm_L10.0mm, Connector_Pin:Pin_D1.0mm_L10.0mm, F.Cu at (188.1, 73.8)
- added REF**: Pin_D1.0mm_L10.0mm, Connector_Pin:Pin_D1.0mm_L10.0mm, F.Cu at (177.9, 86.5)
- added REF**: Pin_D1.0mm_L10.0mm, Connector_Pin:Pin_D1.0mm_L10.0mm, F.Cu at (185.6, 73.8)
- added REF**: Pin_D1.0mm_L10.0mm, Connector_Pin:Pin_D1.0mm_L10.0mm, F.Cu at (183.0, 73.8)
- added REF**: Pin_D1.0mm_L10.0mm, Connector_Pin:Pin_D1.0mm_L10.0mm, F.Cu at (180.5, 73.8)
- added REF**: Pin_D1.0mm_L10.0mm, Connector_Pin:Pin_D1.0mm_L10.0mm, F.Cu at (177.9, 73.8)
- added REF**: Pin_D1.0mm_L10.0mm, Connector_Pin:Pin_D1.0mm_L10.0mm, F.Cu at (175.4, 73.8)
- added REF**: Pin_D1.0mm_L10.0mm, Connector_Pin:Pin_D1.0mm_L10.0mm, F.Cu at (172.9, 73.8)
- added REF**: Pin_D1.0mm_L10.0mm, Connector_Pin:Pin_D1.0mm_L10.0mm, F.Cu at (170.3, 73.8)
- added REF**: Pin_D1.0mm_L10.0mm, Connector_Pin:Pin_D1.0mm_L10.0mm, F.Cu at (167.8, 73.8)
- added REF**: Pin_D1.0mm_L10.0mm, Connector_Pin:Pin_D1.0mm_L10.0mm, F.Cu at (165.2, 73.8)
- added REF**: Pin_D1.0mm_L10.0mm, Connector_Pin:Pin_D1.0mm_L10.0mm, F.Cu at (162.7, 73.8)
- added REF**: Pin_D1.0mm_L10.0mm, Connector_Pin:Pin_D1.0mm_L10.0mm, F.Cu at (175.4, 86.5)
- added REF**: Pin_D1.0mm_L10.0mm, Connector_Pin:Pin_D1.0mm_L10.0mm, F.Cu at (160.2, 73.8)
- added REF**: Pin_D1.0mm_L10.0mm, Connector_Pin:Pin_D1.0mm_L10.0mm, F.Cu at (195.7, 71.2)
- added REF**: Pin_D1.0mm_L10.0mm, Connector_Pin:Pin_D1.0mm_L10.0mm, F.Cu at (193.2, 71.2)
- added REF**: Pin_D1.0mm_L10.0mm, Connector_Pin:Pin_D1.0mm_L10.0mm, F.Cu at (190.6, 71.2)
- added REF**: Pin_D1.0mm_L10.0mm, Connector_Pin:Pin_D1.0mm_L10.0mm, F.Cu at (188.1, 71.2)
- added REF**: Pin_D1.0mm_L10.0mm, Connector_Pin:Pin_D1.0mm_L10.0mm, F.Cu at (185.6, 71.2)
- added REF**: Pin_D1.0mm_L10.0mm, Connector_Pin:Pin_D1.0mm_L10.0mm, F.Cu at (183.0, 71.2)
- added REF**: Pin_D1.0mm_L10.0mm, Connector_Pin:Pin_D1.0mm_L10.0mm, F.Cu at (180.5, 71.2)
- added REF**: Pin_D1.0mm_L10.0mm, Connector_Pin:Pin_D1.0mm_L10.0mm, F.Cu at (177.9, 71.2)
- added REF**: Pin_D1.0mm_L10.0mm, Connector_Pin:Pin_D1.0mm_L10.0mm, F.Cu at (175.4, 71.2)
- C10, C13, C24, C25, C4, C7, D1, D17, D18, D2, D20, D3, D4, D5, D6, Q2, Q3, R1, R10, R11, R12, R13, R14, R2, R29, R3, R30, R32, R35, R39, R4, R47, R48, R49, R5, R50, R6, R7, R8, R9, U1, U2, U6, U7: moved to F.Cu
- C19: footprint Capacitor_SMD:C_0805_2012Metric -> Capacitor_SMD:C_0805_2012Metric_Pad1.15x1.40mm_HandSolder
- JP6, JP7, JP9: moved to B.Cu
- S1: footprint SamacSys_Parts_github:AYZ0202AGRLC -> Misc:AYZ0202AGRLC
- U5: footprint Connector_PinHeader_2.54mm:PinHeader_1x06_P2.54mm_Horizontal -> Misc:MPX4250
- XA1: footprint Arduino:Arduino_Mega2560_Shield -> Shields:Arduino_Mega2560_Shield_IO_Only
- moved D13 234.6 mm to (191.9, 109.0), turned to 180 degrees
- moved R37 222.7 mm to (172.1, 115.0), turned to 270 degrees
- moved R33 202.5 mm to (145.6, 118.7), turned to 180 degrees
- moved C5 191.7 mm to (145.6, 116.6)
- moved C6 171.1 mm to (154.3, 131.4)
- moved R31 161.3 mm to (148.2, 131.4), turned to 180 degrees
- moved C3 159.1 mm to (141.2, 131.4)
- moved Q1 140.6 mm to (153.1, 110.3), turned to 270 degrees
- moved R51 139.0 mm to (155.9, 110.3), turned to 90 degrees
- moved R60 109.4 mm to (159.9, 52.6), turned to 90 degrees
- moved RV1 108.8 mm to (196.8, 51.4)
- moved C18 105.4 mm to (192.3, 51.5), turned to 0 degrees
- moved C17 103.9 mm to (192.8, 45.5), turned to 90 degrees
- moved D14 97.2 mm to (186.5, 48.8), turned to 0 degrees
- moved J3 90.7 mm to (205.0, 49.0), turned to 90 degrees
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Connections:
- A1 pad 10: unconnected-(A1-Pad10) -> Net-(A1-Pad10)
- A1 pad 11: unconnected-(A1-Pad11) -> Net-(A1-Pad11)
- A1 pad 12: unconnected-(A1-Pad12) -> Net-(A1-Pad12)
- A1 pad 2: unconnected-(A1-Pad2) -> Net-(A1-Pad2)
- J2 pad 6: unconnected-(J2-Pad6) -> Net-(J2-Pad6)
- S1 pad 4: unconnected-(S1-Pad4) -> Net-(S1-Pad4)
- S1 pad 5: unconnected-(S1-Pad5) -> Net-(S1-Pad5)
- S1 pad 6: unconnected-(S1-Pad6) -> Net-(S1-Pad6)
- U1 pad 2: unconnected-(U1-Pad2) -> Net-(U1-Pad2)
- U1 pad 4: unconnected-(U1-Pad4) -> Net-(U1-Pad4)
- U2 pad 1: unconnected-(U2-Pad1) -> Net-(U2-Pad1)
- U2 pad 8: unconnected-(U2-Pad8) -> Net-(U2-Pad8)
- U3 pad 2: unconnected-(U3-Pad2) -> Net-(U3-Pad2)
- U3 pad 4: unconnected-(U3-Pad4) -> Net-(U3-Pad4)
- U4 pad 1: unconnected-(U4-Pad1) -> Net-(U4-Pad1)
- U4 pad 8: unconnected-(U4-Pad8) -> Net-(U4-Pad8)
- U7 pad 2: unconnected-(U7-Pad2) -> Net-(U7-Pad2)
- U7 pad 4: unconnected-(U7-Pad4) -> Net-(U7-Pad4)
- U9 pad 2: unconnected-(U9-Pad2) -> Net-(U9-Pad2)
- U9 pad 4: unconnected-(U9-Pad4) -> Net-(U9-Pad4)
- XA1 pad 3V3: unconnected-(XA1-Pad3V3) -> Net-(XA1-Pad3V3)
- XA1 pad A11: unconnected-(XA1-PadA11) -> Net-(XA1-PadA11)
- XA1 pad A12: unconnected-(XA1-PadA12) -> Net-(XA1-PadA12)
- XA1 pad A13: unconnected-(XA1-PadA13) -> Net-(XA1-PadA13)
- XA1 pad A14: unconnected-(XA1-PadA14) -> Net-(XA1-PadA14)
- XA1 pad A15: unconnected-(XA1-PadA15) -> Net-(XA1-PadA15)
- XA1 pad AREF: unconnected-(XA1-PadAREF) -> Net-(XA1-PadAREF)
- XA1 pad IORF: unconnected-(XA1-PadIORF) -> Net-(XA1-PadIORF)
- XA1 pad SCL: unconnected-(XA1-PadSCL) -> Net-(XA1-PadSCL)
- XA1 pad SDA: unconnected-(XA1-PadSDA) -> Net-(XA1-PadSDA)
- XA1 pad VIN: unconnected-(XA1-PadVIN) -> Net-(XA1-PadVIN)
Routing:
- net VDD: track 28.0 -> 347.1 mm, vias 0 -> 5
- net 12V-SW: track 25.7 -> 269.2 mm, vias 0 -> 4
- net ADC-Clamp-10: track 0.00 -> 201.7 mm, vias 0 -> 4
- net VDDA: track 4.67 -> 136.4 mm
- net ADC-Clamp-8: track 20.1 -> 145.2 mm, vias 0 -> 1
- net ADC-Clamp-9: track 12.7 -> 126.3 mm, vias 0 -> 1
- net VR2-: track 0.00 -> 84.8 mm, vias 0 -> 1
- net VR1-: track 0.00 -> 77.9 mm, vias 0 -> 1
- net CRANK-IN: track 4.31 -> 75.5 mm, vias 0 -> 2
- net MCU-D47: track 0.00 -> 69.0 mm, vias 0 -> 1
- net MCU-D45: track 0.00 -> 66.2 mm, vias 0 -> 1
- net Net-(JP11-Pad2): track 4.76 -> 70.3 mm, vias 0 -> 1
- net CAM-IN: track 4.21 -> 66.7 mm, vias 0 -> 2
- net MCU-D24: track 0.00 -> 61.8 mm, vias 0 -> 1
- net Net-(R6-Pad1): track 2.23 -> 64.0 mm
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- added copper zone on B.Cu, net GND
- added copper zone on F.Cu, net GND
Other:
- board size 121.8 x 77.2 mm -> 100 x 100 mm
- net class Default added: clearance 0.2, trace_width 0.25, via_dia 0.8, via_drill 0.4
- board text added: "1"
- board text added: "12V"
- board text added: "2"
- board text added: "3"
- board text added: "4"
- board text added: "5V"
- board text added: "A10"
- board text added: "A9"
- board text added: "ALIGN"
- board text added: "BLUETOOTH"
- board text added: "D21"
- board text added: "DIRECT/TSC"
- board text added: "GND"
- board text added: "IGNITER"
- board text added: "IGNITION CHANNEL"
- board text added: "INJECTOR CHANNEL"
- board text added: "MODULE CHIP THIS END"
- board text added: "MOUNT FLAT SIDE UP"
- board text added: "PRIMARY"
- board text added: "PULL -UP"
- board text added: "Prog"
- board text added: "RESET CONTROL"
- board text added: "RX"
- board text added: "Run"
- board text added: "SECONDARY"
- board text added: "STEPPER IDLE DRV8825"
- board text added: "Speeduino Community"
- board text added: "Speeduino v0.4.4c"
- board text added: "TRIGGER SETUP"
- board text added: "TRIGGER SIGNAL CONDITIONER SOCKET"
- board text added: "TX"
- board text added: "VSS"
- board text added: "© Josh Stewart &"
