File: v0.5/Interface boards/Molex_48/Molex_48/Molex_48.kicad_sch (KiCad schematic)
At the start: 2 parts, among them J1 Conn_02x20_Counter_Clockwise, J2 500762-0482

Commit message: update
Parts:
- added J3, J4: Conn_02x12_Counter_Clockwise, Connector_PinHeader_2.54mm:PinHeader_2x12_P2.54mm_Vertical, symbol Connector_Generic:Conn_02x12_Counter_Clockwise
- J1: now left out of the parts list
Connections:
- net GND: now also J3.1 (Pin_1), J3.10 (Pin_10), J3.2 (Pin_2), J3.3 (Pin_3), J3.4 (Pin_4), J3.7 (Pin_7), J3.8 (Pin_8), J3.9 (Pin_9), J4.1 (Pin_1), J4.10 (Pin_10), J4.2 (Pin_2), J4.3 (Pin_3), J4.4 (Pin_4), J4.7 (Pin_7), J4.8 (Pin_8), J4.9 (Pin_9)
