File: integrated_mcu/V0.1/V0.1.kicad_sch (KiCad schematic)
At the start: 0 parts

Commit message: updates!
Other:
- added sheet injectors_and_coils (injectors_and_coils.kicad_sch)
- added sheet inputs (inputs.kicad_sch)
- added sheet mcu (mcu.kicad_sch)
- added sheet outputs (outputs.kicad_sch)
