File: integrated_mcu/V0.1/alim.kicad_sch (KiCad schematic)
At the start: 3 parts

Commit message: updates!
Parts:
- added C2, C3: 1μF, Capacitor_SMD:C_1206_3216Metric, symbol Device:C
- added C5: 10μF, Capacitor_SMD:C_1206_3216Metric, symbol Device:C
- added C6, C7: C, Capacitor_SMD:C_1206_3216Metric, symbol Device:C
- added D1, D2: D, symbol Device:D
- added D3: 5.6V, symbol Device:D_Schottky
- added D8: 18V, symbol Device:D_Schottky
- added IC1: TPS54225TPWPRQ1, SOP65P640X120-15N, symbol TPS54225TPWPRQ1:TPS54225TPWPRQ1
- added J1: USB_B, symbol Connector:USB_B
- added L1: L, symbol Device:L
- added R1, R2: R, symbol Device:R
- gave numbers to parts that had none: 3
Connections:
- net +12V: now also C5.2, D8.1 (K), IC1.13 (VIN), IC1.14 (VCC), R1.1
- net GND: now also C2.1, C3.1, C5.1, C7.1, D3.2 (A), D8.2 (A), IC1.15 (EP), IC1.5 (GND), IC1.8 (PGND1), IC1.9 (PGND2), J1.4 (GND), J1.5 (Shield), R2.2
- new net: C2.2, IC1.3 (VREG5)
- new net: C6.1, IC1.12 (VBST)
- new net: C6.2, IC1.10 (SW1), IC1.11 (SW2), L1.2
- new net: C3.2, IC1.4 (SS)
- new net: IC1.2 (VFB), R1.2, R2.1
- new net: D1.2 (A), J1.1 (VBUS)
- new net +5P: C7.2, D2.2 (A), IC1.1 (VO), L1.1
- new net +5V: D1.1 (K), D2.1 (K), D3.1 (K)
- new net D+: J1.3 (D+)
- new net D-: J1.2 (D-)
- new net EN: IC1.7 (EN)
- new net PWRGD: IC1.6 (PG)
